File: PCB/MCU Datalogger/MCU Datalogger.kicad_sch (KiCad schematic)
At the start: 25 parts, among them U1 24LC1025, U2 24LC1025, U3 DS1337S+, U4 ATMEGA328P-AU, Y1 16 MHz, Y2 32.768 Khz

Commit message: added comments
Other:
- note added: "EEPROM"
- note added: "MCU"
- note added: "Mounting"
- note added: "Real Time Clock"
- moved on the sheet: H1, H2, H3, H4
Changed lines of the file:
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@@
+    (stroke (width 0) (type default))
+  )
+  (polyline (pts (xy 245.11 160.02) (xy 245.11 115.57))
+    (stroke (width 0) (type default))
+  )
+  (polyline (pts (xy 134.62 101.6) (xy 134.62 20.32))
     (stroke (width 0) (type default))
   )
@@
     (stroke (width 0) (type default))
   )
+  (polyline (pts (xy 16.51 25.4) (xy 16.51 86.36))
+    (stroke (width 0) (type default))
+  )
   (wire (pts (xy 111.76 142.24) (xy 111.76 144.78))
     (stroke (width 0) (type default))
   )
+  (polyline (pts (xy 34.29 156.21) (xy 34.29 116.84))
+    (stroke (width 0) (type default))
+  )
+  (polyline (pts (xy 16.51 25.4) (xy 124.46 25.4))
+    (stroke (width 0) (type default))
+  )
   (wire (pts (xy 121.92 125.73) (xy 121.92 134.62))
     (stroke (width 0) (type default))
@@
     (stroke (width 0) (type default))
   )
+  (polyline (pts (xy 34.29 116.84) (xy 134.62 116.84))
+    (stroke (width 0) (type default))
+  )
   (wire (pts (xy 80.01 138.43) (xy 76.2 138.43))
     (stroke (width 0) (type default))
@@
     (stroke (width 0) (type default))
   )
+  (polyline (pts (xy 276.86 101.6) (xy 134.62 101.6))
+    (stroke (width 0) (type default))
+  )
   (wire (pts (xy 74.93 49.53) (xy 74.93 38.1))
     (stroke (width 0) (type default))
@@
     (stroke (width 0) (type default))
   )
+  (polyline (pts (xy 124.46 86.36) (xy 16.51 86.36))
+    (stroke (width 0) (type default))
+  )
+  (polyline (pts (xy 273.05 115.57) (xy 273.05 160.02))
+    (stroke (width 0) (type default))
+  )
   (wire (pts (xy 116.84 125.73) (xy 121.92 125.73))
     (stroke (width 0) (type default))
@@
     (stroke (width 0) (type default))
   )
+  (polyline (pts (xy 134.62 156.21) (xy 34.29 156.21))
+    (stroke (width 0) (type default))
+  )
+  (polyline (pts (xy 273.05 160.02) (xy 245.11 160.02))
+    (stroke (width 0) (type default))
+  )
   (wire (pts (xy 224.79 85.09) (xy 224.79 87.63))
     (stroke (width 0) (type default))
   )
+  (polyline (pts (xy 245.11 115.57) (xy 273.05 115.57))
+    (stroke (width 0) (type default))
+  )
   (wire (pts (xy 78.74 59.69) (xy 100.33 59.69))
     (stroke (width 0) (type default))
@@
     (stroke (width 0) (type default))
   )
+  (polyline (pts (xy 134.62 20.32) (xy 276.86 20.32))
+    (stroke (width 0) (type default))
+  )
   (wire (pts (xy 163.83 54.61) (xy 175.26 54.61))
     (stroke (width 0) (type default))
@@
     (stroke (width 0) (type default))
   )
+  (polyline (pts (xy 124.46 25.4) (xy 124.46 86.36))
+    (stroke (width 0) (type default))
+  )
   (wire (pts (xy 224.79 36.83) (xy 229.87 36.83))
     (stroke (width 0) (type default))
@@
     (stroke (width 0) (type default))
   )
+  (polyline (pts (xy 276.86 20.32) (xy 276.86 101.6))
+    (stroke (width 0) (type default))
+  )
   (wire (pts (xy 180.34 54.61) (xy 175.26 54.61))
     (stroke (width 0) (type default))
@@
     (stroke (width 0) (type default))
   )
+  (polyline (pts (xy 134.62 116.84) (xy 134.62 156.21))
+    (stroke (width 0) (type default))
+  )
   (wire (pts (xy 67.31 140.97) (xy 67.31 146.05))
     (stroke (width 0) (type default))
@@
   (wire (pts (xy 87.63 38.1) (xy 100.33 38.1))
     (stroke (width 0) (type default))
+  )
+  (text "EEPROM" (at 34.29 115.57 0)
+    (effects (font (size 1.27 1.27)) (justify left bottom))
+  )
+  (text "Mounting" (at 245.11 114.3 0)
+    (effects (font (size 1.27 1.27)) (justify left bottom))
+  )
+  (text "MCU" (at 134.62 19.05 0)
+    (effects (font (size 1.27 1.27)) (justify left bottom))
+  )
+  (text "Real Time Clock" (at 16.51 24.13 0)
+    (effects (font (size 1.27 1.27)) (justify left bottom))
   )
   (label "Vcc" (at 46.99 140.97 180) (fields_autoplaced)
@@
     )
   )
-  (symbol (lib_id "Mechanical:MountingHole") (at 261.62 158.75 0) (unit 1)
-    (in_bom yes) (on_board yes) (dnp no) (fields_autoplaced)
-    (property "Reference" "H4" (at 264.16 157.48 0)
-      (effects (font (size 1.27 1.27)) (justify left))
-    )
-    (property "Value" "MountingHole" (at 264.16 160.02 0)
-      (effects (font (size 1.27 1.27)) (justify left))
-    )
-    (property "Footprint" "MountingHole:MountingHole_2.1mm" (at 261.62 158.75 0)
-      (effects (font (size 1.27 1.27)) hide)
-    )
-    (property "Datasheet" "~" (at 261.62 158.75 0)
+  (symbol (lib_id "Mechanical:MountingHole") (at 252.73 153.67 0) (unit 1)
+    (in_bom yes) (on_board yes) (dnp no) (fields_autoplaced)
+    (property "Reference" "H4" (at 255.27 152.4 0)
+      (effects (font (size 1.27 1.27)) (justify left))
+    )
+    (property "Value" "MountingHole" (at 255.27 154.94 0)
+      (effects (font (size 1.27 1.27)) (justify left))
+    )
+    (property "Footprint" "MountingHole:MountingHole_2.1mm" (at 252.73 153.67 0)
+      (effects (font (size 1.27 1.27)) hide)
+    )
+    (property "Datasheet" "~" (at 252.73 153.67 0)
       (effects (font (size 1.27 1.27)) hide)
     )
@@
     )
   )
-  (symbol (lib_id "Mechanical:MountingHole") (at 260.35 147.32 0) (unit 1)
-    (in_bom yes) (on_board yes) (dnp no) (fields_autoplaced)
-    (property "Reference" "H3" (at 262.89 146.05 0)
-      (effects (font (size 1.27 1.27)) (justify left))
-    )
-    (property "Value" "MountingHole" (at 262.89 148.59 0)
-      (effects (font (size 1.27 1.27)) (justify left))
-    )
-    (property "Footprint" "MountingHole:MountingHole_2.1mm" (at 260.35 147.32 0)
-      (effects (font (size 1.27 1.27)) hide)
-    )
-    (property "Datasheet" "~" (at 260.35 147.32 0)
+  (symbol (lib_id "Mechanical:MountingHole") (at 251.46 142.24 0) (unit 1)
+    (in_bom yes) (on_board yes) (dnp no) (fields_autoplaced)
+    (property "Reference" "H3" (at 254 140.97 0)
+      (effects (font (size 1.27 1.27)) (justify left))
+    )
+    (property "Value" "MountingHole" (at 254 143.51 0)
+      (effects (font (size 1.27 1.27)) (justify left))
+    )
+    (property "Footprint" "MountingHole:MountingHole_2.1mm" (at 251.46 142.24 0)
+      (effects (font (size 1.27 1.27)) hide)
+    )
+    (property "Datasheet" "~" (at 251.46 142.24 0)
       (effects (font (size 1.27 1.27)) hide)
     )
@@
     )
   )
-  (symbol (lib_id "Mechanical:MountingHole") (at 260.35 128.27 0) (unit 1)
-    (in_bom yes) (on_board yes) (dnp no) (fields_autoplaced)
-    (property "Reference" "H1" (at 262.89 127 0)
-      (effects (font (size 1.27 1.27)) (justify left))
-    )
-    (property "Value" "MountingHole" (at 262.89 129.54 0)
-      (effects (font (size 1.27 1.27)) (justify left))
-    )
-    (property "Footprint" "MountingHole:MountingHole_2.1mm" (at 260.35 128.27 0)
-      (effects (font (size 1.27 1.27)) hide)
-    )
-    (property "Datasheet" "~" (at 260.35 128.27 0)
+  (symbol (lib_id "Mechanical:MountingHole") (at 251.46 123.19 0) (unit 1)
+    (in_bom yes) (on_board yes) (dnp no) (fields_autoplaced)
+    (property "Reference" "H1" (at 254 121.92 0)
+      (effects (font (size 1.27 1.27)) (justify left))
+    )
+    (property "Value" "MountingHole" (at 254 124.46 0)
+      (effects (font (size 1.27 1.27)) (justify left))
+    )
+    (property "Footprint" "MountingHole:MountingHole_2.1mm" (at 251.46 123.19 0)
+      (effects (font (size 1.27 1.27)) hide)
+    )
+    (property "Datasheet" "~" (at 251.46 123.19 0)
       (effects (font (size 1.27 1.27)) hide)
     )
@@
     )
   )
-  (symbol (lib_id "Mechanical:MountingHole") (at 260.35 137.16 0) (unit 1)
-    (in_bom yes) (on_board yes) (dnp no) (fields_autoplaced)
-    (property "Reference" "H2" (at 262.89 135.89 0)
-      (effects (font (size 1.27 1.27)) (justify left))
-    )
-    (property "Value" "MountingHole" (at 262.89 138.43 0)
-      (effects (font (size 1.27 1.27)) (justify left))
-    )
-    (property "Footprint" "MountingHole:MountingHole_2.1mm" (at 260.35 137.16 0)
-      (effects (font (size 1.27 1.27)) hide)
-    )
-    (property "Datasheet" "~" (at 260.35 137.16 0)
-      (effects (font (size 1.27 1.27)) hide)
-    )
+  (symbol (lib_id "Mechanical:MountingHole") (at 251.46 132.08 0) (unit 1)
+    (in_bom yes) (on_board yes) (dnp no) (fields_autoplaced)
+    (property "Reference" "H2" (at 254 130.81 0)
+      (effects (font (size 1.27 1.27)) (justify left))
+    )
+    (property "Value" "MountingHole" (at 254 133.35 0)
+      (effects (font (size 1.27 1.27)) (justify left))
+    )
+    (property "Footprint" "MountingHole:MountingHole_2.1mm" (at 251.46 132.08 0)
+      (effects (font (size 1.27 1.27)) hide)
+    )
+    (property "Datasheet" "~" (at 251.46 132.08 0)
+      (effects (font (size 1.27 1.27)) hide)
+    )
