File: PCB/MCU Datalogger - 2 Layer/MCU Datalogger.kicad_pcb (KiCad board)
At the start: 2 copper layers, 29 parts, among them J1 Conn_01x04_Pin, J2 Conn_01x04_Pin, J3 Conn_01x09_Pin, J4 Conn_02x03_Odd_Even, U1 24LC1025, U2 24LC1025, U3 DS1337S+, U4 ATMEGA328P-AU, Y1 16 MHz, Y2 32.768 Khz

Commit message: placed components
Parts:
- R1, R2, R3, R4, R5, R6, R7: footprint Resistor_SMD:R_0815_2038Metric -> Resistor_SMD:R_0805_2012Metric
- moved J3 47.9 mm to (131.0, 115.3), turned to 90 degrees
- moved H4 43.0 mm to (171.6, 115.9)
- moved J2 42.9 mm to (155.4, 115.4), turned to 90 degrees
- moved R1 42.3 mm to (156.8, 95.3)
- moved R2 42.3 mm to (161.3, 95.3)
- moved H3 38.5 mm to (171.6, 90.5)
- moved R3 36.9 mm to (132.9, 110.5), turned to 180 degrees
- moved R4 36.9 mm to (136.9, 110.5), turned to 180 degrees
- moved R5 34.9 mm to (156.8, 103.4), turned to 180 degrees
- moved J1 32.0 mm to (168.4, 103.9)
- moved H2 31.5 mm to (125.9, 115.9)
- moved Y1 30.6 mm to (147.5, 108.9)
- moved C1 29.6 mm to (156.6, 111.0), turned to 180 degrees
- moved R6 29.5 mm to (156.8, 99.7), turned to 180 degrees
- moved R7 29.5 mm to (161.3, 99.7)
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Other:
- board outline added: 50.8 x 30.5 mm

Commit message: Route
Parts:
- moved J2 2.57 mm to (157.7, 114.4)
- moved D2 1.78 mm to (162.8, 91.7)
- moved J4 1.63 mm to (167.5, 95.0)
- moved J1 1.63 mm to (170.1, 103.9)
- moved R2 1.55 mm to (162.8, 95.3), turned to 180 degrees
- moved R7 1.55 mm to (162.8, 99.7)
- moved D1 1.54 mm to (158.0, 91.8)
- moved C3 1.49 mm to (148.2, 91.8)
- moved U1 1.46 mm to (135.6, 100.6)
- moved U2 1.46 mm to (135.6, 93.6)
- moved U3 1.46 mm to (136.0, 106.9)
- moved C5 1.31 mm to (153.0, 91.8)
- moved C4 1.30 mm to (143.1, 91.8)
- moved R4 1.09 mm to (137.8, 111.2)
- moved R3 1.09 mm to (133.7, 111.2), turned to 0 degrees
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Connections:
- R5 pad 1: Net-(R5-Pad1) -> /Vcc
- R6 pad 1: Net-(R5-Pad1) -> /Vcc
Routing:
- net /Vcc: track 0.00 -> 102.5 mm, vias 0 -> 1
- net /SCK: track 0.00 -> 102.3 mm, vias 0 -> 4
- net /RX: track 0.00 -> 72.8 mm, vias 0 -> 1
- net Net-(BT1-+): track 0.00 -> 67.0 mm, vias 0 -> 4
- net /SDA: track 0.00 -> 60.5 mm, vias 0 -> 2
- net GND: track 0.00 -> 50.1 mm, vias 0 -> 6
- net /TX: track 0.00 -> 32.0 mm, vias 0 -> 1
- net Net-(U4-PB7): track 0.00 -> 30.5 mm, vias 0 -> 2
- net /D2: track 0.00 -> 29.2 mm, vias 0 -> 1
- net /D3: track 0.00 -> 27.2 mm
- net /D4: track 0.00 -> 26.5 mm
- net /MOSI: track 0.00 -> 25.7 mm
- net /D8: track 0.00 -> 24.9 mm, vias 0 -> 1
- net /RESET: track 0.00 -> 24.2 mm, vias 0 -> 2
- net Net-(U4-PB6): track 0.00 -> 23.5 mm
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Other:
- board size 50.8 x 30.5 mm -> 50.7 x 30.4 mm
