File: PCB/MCU Datalogger - 2 Layer/MCU Datalogger.kicad_sch (KiCad schematic)
At the start: 25 parts, among them U1 24LC1025, U2 24LC1025, U3 DS1337S+, U4 ATMEGA328P-AU, Y1 16 MHz, Y2 32.768 Khz

Commit message: placed components
Parts:
- R1, R2, R3, R4, R5, R6, R7: footprint Resistor_SMD:R_0815_2038Metric -> Resistor_SMD:R_0805_2012Metric
Changed lines of the file:
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@@
       (effects (font (size 1.27 1.27)) (justify left))
     )
-    (property "Footprint" "Resistor_SMD:R_0815_2038Metric" (at 98.552 53.34 90)
+    (property "Footprint" "Resistor_SMD:R_0805_2012Metric" (at 98.552 53.34 90)
       (effects (font (size 1.27 1.27)) hide)
     )
@@
       (effects (font (size 1.27 1.27)) (justify left))
     )
-    (property "Footprint" "Resistor_SMD:R_0815_2038Metric" (at 120.142 138.43 90)
+    (property "Footprint" "Resistor_SMD:R_0805_2012Metric" (at 120.142 138.43 90)
       (effects (font (size 1.27 1.27)) hide)
     )
@@
       (effects (font (size 1.27 1.27)) (justify left))
     )
-    (property "Footprint" "Resistor_SMD:R_0815_2038Metric" (at 85.852 53.34 90)
+    (property "Footprint" "Resistor_SMD:R_0805_2012Metric" (at 85.852 53.34 90)
       (effects (font (size 1.27 1.27)) hide)
     )
@@
       (effects (font (size 1.27 1.27)) (justify left))
     )
-    (property "Footprint" "Resistor_SMD:R_0815_2038Metric" (at 109.982 138.43 90)
+    (property "Footprint" "Resistor_SMD:R_0805_2012Metric" (at 109.982 138.43 90)
       (effects (font (size 1.27 1.27)) hide)
     )
@@
       (effects (font (size 1.27 1.27)) (justify left))
     )
-    (property "Footprint" "Resistor_SMD:R_0815_2038Metric" (at 235.712 68.58 90)
+    (property "Footprint" "Resistor_SMD:R_0805_2012Metric" (at 235.712 68.58 90)
       (effects (font (size 1.27 1.27)) hide)
     )
@@
       (effects (font (size 1.27 1.27)))
     )
-    (property "Footprint" "Resistor_SMD:R_0815_2038Metric" (at 160.02 43.688 90)
+    (property "Footprint" "Resistor_SMD:R_0805_2012Metric" (at 160.02 43.688 90)
       (effects (font (size 1.27 1.27)) hide)
     )
@@
       (effects (font (size 1.27 1.27)))
     )
-    (property "Footprint" "Resistor_SMD:R_0815_2038Metric" (at 182.88 84.328 90)
-      (effects (font (size 1.27 1.27)) hide)
-    )
+    (property "Footprint" "Resistor_SMD:R_0805_2012Metric" (at 182.88 84.328 90)
+      (effects (font (size 1.27 1.27)) hide)
+    )

Commit message: Route
Connections:
- net Vcc: now also R5.1, R6.1
Changed lines of the file:
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@@
+    (effects (font (size 1.27 1.27)) (justify right bottom))
+  )
+  (label "Vcc" (at 116.84 121.92 180) (fields_autoplaced)
     (effects (font (size 1.27 1.27)) (justify right bottom))
   )
